File: KiCad/proj_Checkpoint2/_autosave-proj_Checkpoint1.kicad_sch (KiCad schematic)
At the start: 37 parts, among them M1 Motor_Servo, Q2 MOSFET-N, SW1 Reset, U1 74xxx244, U1 MCP6294, U1 PIC32MX170F256B, U2 Comparator, U5 SW_CapTouch, U8 LED_Matrix

Commit message: update
Other:
- note added: "Coin Detector IR"
- note added: "Goal Sensor IR"
- note added: "Miss Sensor"
Changed lines of the file:
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@@
     (effects (font (size 1.27 1.27)) (justify left bottom))
   )
-  (text "IR Sensor Signal Regulator\n" (at 106.68 171.45 0)
+  (text "Coin Detector IR" (at 106.68 171.45 0)
     (effects (font (size 1.27 1.27)) (justify left bottom))
   )
-  (text "IR Sensor Signal Regulator\n" (at 106.68 189.23 0)
+  (text "Goal Sensor IR\n" (at 106.68 189.23 0)
     (effects (font (size 1.27 1.27)) (justify left bottom))
   )
@@
     (effects (font (size 1.27 1.27)) (justify left bottom))
   )
-  (text "IR Sensor Signal Regulator\n" (at 106.68 180.34 0)
+  (text "Miss Sensor" (at 106.68 180.34 0)
     (effects (font (size 1.27 1.27)) (justify left bottom))
   )
